File: TXV2/kicad/revB/TXV2_MAIN_revB.kicad_pcb (KiCad board)
At the start: 4 copper layers, 83.3 x 91.7 mm, 64 parts, among them J1 USB-C, J10 TRIMS, J11 RGB LED, J12 QWIIC, J13 I2C, J14 RTC, J15 ESP-A, J16 ESP-B, J17 TX MODULE, J2 NEXTION, J3 BATT, J4 BAL, J5 BTN, J6 GIM R V, J6B GIM R H, J7 GIM L V, J7B GIM L H, J8 KNOBS, J9 SWITCHES, U1 Teensy 4.1, U2 ESP32-S3-DevKitC, U3 nRF24L01, U4 Pololu 2808, U5 5V buck MAIN, U7 BQ25887, U8 AMS1117-3.3, U9 5V buck NEXT

Commit message: TXV2 Rev-B: silkscreen clarity pass (bigger labels, 2808 pin names, C12/SS14/pin-1 marks, labels off pads)
Co-Authored-By: Claude Fable 5.1 <noreply@anthropic.com>
Claude-Session: https://claude.ai/code/session_01DvvNNevU4xtNTYtdVBAM7h
Parts:
- D3, D4: value 1N4001 -> SS14
Other:
- board text added: "2808 right way up"
- board text added: "A"
- board text added: "B"
- board text added: "C12 10uF"
- board text added: "CTRL"
- board text added: "OFF"
- board text added: "ON"
- board text added: "VIN"
- board text added: "VOUT"
- board text added: "by Claude and Malcolm - 2026"
- board text added: "microSD end ^"
- board text removed: "2808 right way up, VIN row at the bottom"
- board text removed: "by Claude and Malcolm - July 2026"
- board text removed: "microSD exits ^ (top edge)"
